File: deplacement_2019_f103.kicad_pcb (KiCad board)
At the start: 2 copper layers, 52.1 x 87 mm, 30 parts, among them J1 Alim logique, J2 Connecteur Gauche, J3 Connecteur Droit, J4 Conn_01x05, J5 Conn_01x05, J6 PWM output, J7 PWM output, J8 Liaison serie, Q1 PMF370XN, Q2 PMF370XN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

Commit message: Update footprints and board
Parts:
- removed TP1, TP2, TP3, TP4, TP5, TP6: TestPoint_Probe, Connector_PinHeader_1.00mm:PinHeader_1x01_P1.00mm_Vertical
- J1, J6, J7, J8: footprint @Robot:HE14-3-straight -> TerminalBlock_Phoenix:TerminalBlock_Phoenix_MPT-0,5-3-2.54_1x03_P2.54mm_Horizontal
- J4, J5: footprint @Robot:HE14-5-straight -> TerminalBlock_Phoenix:TerminalBlock_Phoenix_MPT-0,5-5-2.54_1x05_P2.54mm_Horizontal
- moved J6 3.51 mm to (110.0, 92.0)
- moved J8 2.50 mm to (138.5, 87.5), turned to 90 degrees
- moved J4 2.48 mm to (110.0, 106.0)
- moved J1 1.44 mm to (110.0, 122.5)
- moved J7 1.37 mm to (138.0, 100.5)
Connections:
- J2 pad 10: Net-(J2-Pad10) -> GND
Routing:
- net /motor_right_PWM: track 35.8 -> 10.4 mm
- net /qei_left_A: track 25.0 -> 8.30 mm
- net /motor_left_direction: track 19.5 -> 7.13 mm
- net /motor_right_direction: track 18.7 -> 30.4 mm
- net /qei_right_A: track 16.9 -> 7.61 mm
- net /motor_left_PWM: track 98.8 -> 91.2 mm
- net /TX: track 6.78 -> 13.9 mm
- net /qei_left_B: track 6.52 -> 7.67 mm
- net +5V: track 150.7 -> 151.4 mm
Other:
- board text added: "deplacement 2019 v1.1 by alex & Paul club robot"
- board text removed: "deplacement 2019 v1 by alex salazar club robot"
